File: Helm.brd (EAGLE design)
At the start: 40.3 x 47.6 mm, 21 parts, among them IC1 DS89C21, IC2 DS89C21, X5 SM06B-SRSS-TB

Commit message: WIP on v2 of the board
Parts:
- removed C1: (no value), SparkFun-Capacitors:0805
- removed Q3, Q4: (no value), SparkFun-DiscreteSemi:SOT23
- removed R1, R2, R4: 10k, SparkFun-Passives:0603-RES
- removed R3: 3.9k, SparkFun-Passives:0603-RES
- removed R6: 15k, SparkFun-Passives:0603-RES
- removed U$1: ARDUINO_PRO_MICRO, SparkFun-Boards:ARDUINO_PRO_MICRO
- added Q1: PMBT3906, SparkFun-DiscreteSemi:SOT23-3
- added Q2: MMBT5088, SparkFun-DiscreteSemi:SOT23-3
- added R10, R7: 15k, SparkFun-Passives:0603-RES
- added R11: 1k, SparkFun-Passives:0603-RES
- added R12: 3.9k, SparkFun-Passives:0603-RES
- added R5: 30k, SparkFun-Passives:0603-RES
- added R8, R9: 2.2k, SparkFun-Passives:0603-RES
- added SJ1: SOLDERJUMPERTRACE, SparkFun-Retired:SJ_2S-TRACE
- added SJ2: SOLDERJUMPERNO, SparkFun-Retired:SJ_2S-NO
- added U$2: TEENSY_3.1_BASIC, Teensy_3_Series_Board_v1.0:TEENSY_3.1_BASIC
Connections:
- removed net N$1: Q4.1, R1.2
- removed net N$4: Q3.1, R3.2, R4.2
- removed net VRAW: C5.1, JP4.2, U$1.24
- new net 3.3V: SJ2.2, U$2.3.3V, U$2.3.3V1
- new net GPS-SUPPLY: C4.1, SJ1.2, SJ2.1, X5.5
- new net N$2: Q1.3, R5.2
- new net N$3: Q1.1, R8.2, R9.1
- new net N$9: Q2.1, R11.1, R12.2
- new net VBAT: U$2.VBAT
- net 5V: now also C5.1, JP4.2, SJ1.1, U$2.VIN; no longer C1.1, C4.1, R2.2, U$1.21, X5.5
- net GND: now also Q2.2, R12.1, R7.1, U$2.AGND, U$2.GND, U$2.GND1; no longer C1.2, Q3.2, Q4.2, R3.1, U$1.23, U$1.3, U$1.4
- net GPS-PWRCTRL: now also U$2.11; no longer U$1.18
- net GPS-RX: now also U$2.9; no longer U$1.17
- net GPS-TX: now also U$2.10; no longer U$1.16
- net NMEA-HS-RX: now also U$2.0; no longer U$1.2
- net NMEA-HS-TX: now also U$2.1; no longer U$1.1
- net NMEA-RX: now also U$2.20/A6; no longer U$1.5
- net NMEA-TX: now also U$2.21/A7; no longer U$1.6
- net SEATALK-12V: now also Q1.2, R10.2, R9.2; no longer R6.2
- net SEATALK-DATA: now also Q2.3, R10.1, R8.1; no longer Q3.3, R1.1, R6.1
- net SEATALK-RX: now also R5.1, R7.2, U$2.7; no longer Q4.3, R2.1, U$1.7
- net SEATALK-TX: now also R11.2, U$2.8; no longer R4.1, U$1.8
Routing:
- net VRAW: track 45.4 -> 0.00 mm, vias 2 -> 0
- net NMEA-TX: track 11.2 -> 27.7 mm
- net GPS-PWRCTRL: track 27.9 -> 11.5 mm
- net 5V: track 107.2 -> 91.5 mm, vias 2 -> 1
- net GPS-SUPPLY: track 0.00 -> 13.5 mm
- net N$4: track 10.1 -> 0.00 mm
- net SEATALK-12V: track 13.9 -> 22.9 mm, vias 0 -> 1
- net GPS-TX: track 21.6 -> 14.1 mm
- net NMEA-RX: track 18.5 -> 25.9 mm
- net N$9: track 0.00 -> 6.53 mm
- net GPS-RX: track 24.6 -> 18.1 mm
- net SEATALK-TX: track 27.4 -> 22.1 mm
- net NMEA-HS-RX: track 7.11 -> 12.3 mm
- net N$3: track 0.00 -> 4.81 mm
- net 3.3V: track 0.00 -> 4.21 mm
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Other:
- board text added: "3.3V"
- board text added: "5V"
- board text added: "GPS Supply"
- board text added: "Helm v2"
- board text removed: "Helm v1"
