File: Helm.sch (EAGLE design)
At the start: 21 parts, among them IC1 DS89C21, IC2 DS89C21, X5 SM06B-SRSS-TB

Commit message: WIP on v2 of the board
Parts:
- removed C1: (no value), SparkFun-Capacitors:CAP0805
- removed Q3, Q4: (no value), SparkFun-DiscreteSemi:TRANSISTOR_NPNSOT23
- removed R1, R2, R4: 10k, SparkFun-Passives:RESISTOR0603-RES
- removed R3: 3.9k, SparkFun-Passives:RESISTOR0603-RES
- removed R6: 15k, SparkFun-Passives:RESISTOR0603-RES
- removed U$1: ARDUINO_PRO_MICRO, SparkFun-Boards:ARDUINO_PRO_MICRO
- added Q1: PMBT3906, SparkFun-DiscreteSemi:TRANSISTOR_PNPPMBT3906
- added Q2: MMBT5088, SparkFun-DiscreteSemi:TRANSISTOR_NPNMMBT5088
- added R10, R7: 15k, SparkFun-Passives:RESISTOR0603-RES
- added R11: 1k, SparkFun-Passives:RESISTOR0603-RES
- added R12: 3.9k, SparkFun-Passives:RESISTOR0603-RES
- added R5: 30k, SparkFun-Passives:RESISTOR0603-RES
- added R8, R9: 2.2k, SparkFun-Passives:RESISTOR0603-RES
- added SJ1: SOLDERJUMPERTRACE, SparkFun-Retired:SOLDERJUMPERTRACE
- added SJ2: SOLDERJUMPERNO, SparkFun-Retired:SOLDERJUMPERNO
- added U$2: TEENSY_3.1_BASIC, Teensy_3_Series_Board_v1.0:TEENSY_3.1_BASIC
Connections:
- removed net N$1: Q4.B, R1.2
- removed net N$4: Q3.B, R3.2, R4.2
- removed net VRAW: C5.1, JP4.2, U$1.RAW
- new net 3.3V: SJ2.2, U$2.3.3V
- new net GPS-SUPPLY: C4.1, SJ1.2, SJ2.1, X5-5.S
- new net N$2: Q1.C, R5.2
- new net N$3: Q1.B, R8.2, R9.1
- new net N$9: Q2.B, R11.1, R12.2
- net 5V: now also C5.1, JP4.2, SJ1.1, U$2.VIN; no longer C1.1, C4.1, R2.2, U$1.VCC, X5-5.S
- net GND: now also Q2.E, R12.1, R7.1, U$2.AGND, U$2.GND; no longer C1.2, Q3.E, Q4.E, R3.1, U$1.GND, U$1.GND@1, U$1.GND@2
- net GPS-PWRCTRL: now also U$2.11/MOSI; no longer U$1.A1
- net GPS-RX: now also U$2.9/RX2/PWM; no longer U$1.A0
- net GPS-TX: now also U$2.10/TX2/PWM; no longer U$1.15(SCK)
- net NMEA-HS-RX: now also U$2.0/RX1/T; no longer U$1.RXI
- net NMEA-HS-TX: now also U$2.1/TX1/T; no longer U$1.TXO
- net NMEA-RX: now also U$2.20/A6/PWM; no longer U$1.2
- net NMEA-TX: now also U$2.21/A7/PWM; no longer U$1.*3
- net SEATALK-12V: now also Q1.E, R10.2, R9.2; no longer R6.2
- net SEATALK-DATA: now also Q2.C, R10.1, R8.1; no longer Q3.C, R1.1, R6.1
- net SEATALK-RX: now also R5.1, R7.2, U$2.7/RX3; no longer Q4.C, R2.1, U$1.4
- net SEATALK-TX: now also R11.2, U$2.8/TX3; no longer R4.1, U$1.*5
Other:
- note added: "Not totally sure why but this was def necessary in testing"
- note added: "Wasn't necessary in testing"
- note added: "maybe 1k?"
- note added: "optional?"
- note removed: "Arduino"
- moved on the sheet: C4, C5, C6
